File: V2/eumesmo-brk-1ch-v2.kicad_sch (KiCad schematic)
At the start: 2 parts, among them J1 RJ45, J2 250-204

Commit message: Adjusted component rotation and offset information for JLCPCB.
Parts:
- J1: FT Position Offset (none) -> 0,1.78; FT Rotation Offset (none) -> 0; JLCPCB BOM 1 -> (none); LCSC Part C385834 -> (none); LCSC Part # (none) -> C385834
- J2: FT Rotation Offset (none) -> 0; JLCPCB BOM 1 -> (none); LCSC Part C2765063 -> (none); LCSC Part # (none) -> C2765063
Changed lines of the file:
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@@
 			)
 		)
-		(property "JLCPCB BOM" "1"
+		(property "LCSC Part #" "C385834"
 			(at 133.35 101.6 0)
 			(hide yes)
@@
 			)
 		)
-		(property "LCSC Part" "C385834"
+		(property "FT Position Offset" "0,1.78"
+			(at 133.35 101.6 0)
+			(hide yes)
+			(show_name no)
+			(do_not_autoplace no)
+			(effects
+				(font
+					(size 1.27 1.27)
+				)
+			)
+		)
+		(property "FT Rotation Offset" "0"
 			(at 133.35 101.6 0)
 			(hide yes)
@@
 			)
 		)
-		(property "JLCPCB BOM" "1"
-			(at 170.18 99.06 0)
-			(hide yes)
-			(show_name no)
-			(do_not_autoplace no)
-			(effects
-				(font
-					(size 1.27 1.27)
-				)
-			)
-		)
-		(property "LCSC Part" "C2765063"
-			(at 170.18 99.06 0)
-			(hide yes)
-			(show_name no)
-			(do_not_autoplace no)
-			(effects
-				(font
-					(size 1.27 1.27)
-				)
-			)
-		)
 		(property "Mfr" "Wago"
 			(at 170.18 99.06 0)
@@
 			(at 170.18 99.06 0)
 			(hide yes)
+			(show_name no)
+			(do_not_autoplace no)
+			(effects
+				(font
+					(size 1.27 1.27)
+				)
+			)
+		)
+		(property "LCSC Part #" "C2765063"
+			(at 170.18 99.06 0)
+			(hide yes)
+			(show_name no)
+			(do_not_autoplace no)
+			(effects
+				(font
+					(size 1.27 1.27)
+				)
+			)
+		)
+		(property "FT Position Offset" ""
+			(at 170.18 99.06 0)
+			(hide yes)
+			(show_name no)
+			(do_not_autoplace no)
+			(effects
+				(font
+					(size 1.27 1.27)
+				)
+			)
+		)
+		(property "FT Rotation Offset" "0"
+			(at 170.18 99.06 0)
+			(hide yes)

Commit message: Replaced Wago connectors for other brand, no stock.
Parts:
- J2: LCSC Part # C2765063 -> C475156; Mfr Wago -> Cixi Kefa Elec; Mfr PN 250-204 -> KF250-3.5-4P-1; Vendor PN C2765063 -> C475156
Changed lines of the file:
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@@
 			)
 		)
-		(property "Mfr" "Wago"
+		(property "Mfr" "Cixi Kefa Elec"
 			(at 170.18 99.06 0)
 			(hide yes)
@@
 			)
 		)
-		(property "Mfr PN" "250-204"
+		(property "Mfr PN" "KF250-3.5-4P-1"
 			(at 170.18 99.06 0)
 			(hide yes)
@@
 			)
 		)
-		(property "Vendor PN" "C2765063"
+		(property "Vendor PN" "C475156"
 			(at 170.18 99.06 0)
 			(hide yes)
@@
 			)
 		)
-		(property "LCSC Part #" "C2765063"
+		(property "LCSC Part #" "C475156"
 			(at 170.18 99.06 0)
 			(hide yes)
